File: GPS_proyect_SIM33ELA.kicad_pcb (KiCad board)
At the start: 4 copper layers, 20 x 56.6 mm, 70 parts, among them J1 U.FL-R-SMT_10_, J2 MICROQTJ, Q1 DTC143ZUAT106, Q2 DTC143ZUAT106, Q3 AO3415, Q4 BSS138, Q5 BSS138, Q6 BSS138, U1 ESP32-C3FH4, U2 SIM33ELA, U3 TP4057, U4 EG800KEULC-I03-SNNSA, U5 DIODES AP2210N-3.3TRG1

Commit message: ultima version
Parts:
- added D6: LED, LED_SMD:LED_0603_1608Metric_Pad1.05x0.95mm_HandSolder, F.Cu at (95.2, 53.8)
- added D7: LED, LED_SMD:LED_0603_1608Metric_Pad1.05x0.95mm_HandSolder, F.Cu at (95.2, 50.4)
- added Q4: DTC143ZUAT106, Package_TO_SOT_SMD:SOT-323_SC-70, B.Cu at (94.2, 53.8)
- added Q5: DTC143ZUAT106, Package_TO_SOT_SMD:SOT-323_SC-70, B.Cu at (94.2, 50.3)
- added R16: 2.2k, Resistor_SMD:R_0603_1608Metric_Pad0.98x0.95mm_HandSolder, F.Cu at (93.7, 53.8)
- added R17: 2.2k, Resistor_SMD:R_0603_1608Metric_Pad0.98x0.95mm_HandSolder, F.Cu at (93.7, 50.4)
- BAT+1, BAT-1: moved to B.Cu
- D2, D3, D4: value KUU SS36 -> D_Shockley
- moved BAT+1 20.0 mm to (78.6, 65.0)
- moved BAT-1 16.9 mm to (78.6, 62.1)
- moved D2 6.30 mm to (90.6, 71.0), turned to 0 degrees
- moved D4 1.78 mm to (87.2, 65.5)
- moved D3 1.69 mm to (87.2, 70.0)
- moved J1 1.64 mm to (93.2, 23.4)
- moved C7 0.88 mm to (94.1, 58.2)
- moved R10 0.88 mm to (94.1, 59.7), turned to 0 degrees
- moved R5 0.88 mm to (94.1, 61.2)
- moved R6 0.88 mm to (94.1, 56.8), turned to 0 degrees
- renumbered C7 to C10, C8 to C11, C9 to C12, C10 to C13, C11 to C14, C12 to C15, C13 to C16, C14 to C17, C15 to C18, C16 to C19, C25 to C2, C17 to C20, C18 to C21, C19 to C22, C20 to C23, C21 to C24, C22 to C25, C23 to C26, C24 to C27, C2 to C3, C26 to C4, C27 to C5, C3 to C6, C4 to C7, C5 to C8, C6 to C9, Q4 to Q6, Q5 to Q7, Q6 to Q8, R9 to R10, R10 to R11, R11 to R12, R12 to R13, R13 to R14, R18 to R15, R14 to R18, R15 to R19, R16 to R20, R17 to R4, R4 to R5, R5 to R6, R6 to R7, R7 to R8, R8 to R9
Connections:
- D2 pad 1: (no net) -> Net-(D2-K)
- D2 pad 2: (no net) -> +5V
- D3 pad 1: (no net) -> Net-(D3-K)
- D3 pad 2: (no net) -> Net-(D2-K)
- D4 pad 1: (no net) -> +4V
- D4 pad 2: (no net) -> Net-(D3-K)
- U2 pad 4: Net-(U2-GND-Pad4) -> GND
- U2 pad 5: Net-(U2-GND-Pad4) -> GND
- U4 pad 16: unconnected-(U4A-NET_STATUS-Pad16) -> /EG800K.NET_STATUS
- U4 pad 25: unconnected-(U4A-STATUS-Pad25) -> /EG800K.STATUS
Routing:
- net /EG800K.VBAT: track 31.8 -> 64.1 mm
- net +4.2V: track 37.8 -> 20.6 mm, vias 8 -> 0
- net /EG800K.NET_STATUS: track 0.00 -> 13.1 mm, vias 0 -> 1
- net /EG800K.STATUS: track 0.00 -> 12.6 mm, vias 0 -> 1
- net /Strapping GPIO9: track 10.8 -> 18.9 mm
- net Net-(Q5-C): track 0.00 -> 5.54 mm, vias 0 -> 1
- net GND: track 59.1 -> 64.6 mm, vias 352 -> 308
- net Net-(Q4-C): track 0.00 -> 5.44 mm, vias 0 -> 1
- net +4V: track 98.3 -> 103.1 mm
- net +5V: track 15.6 -> 18.7 mm
- net (no net): track 2.72 -> 0.00 mm
- net Net-(D2-K): track 0.00 -> 2.09 mm
- net /RF_ANT: track 3.69 -> 5.32 mm
- net /Strapping GPIO8: track 3.46 -> 5.06 mm
- net Net-(D3-K): track 0.00 -> 1.60 mm
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Other:
- board text added: "+ -"
- board text added: "JLC04161H-7628"
- board text added: "NET"
- board text added: "STA"
- board text removed: "JLC04161H-7628(Standard/Finished thickness1.59mm"
