File: GPS_proyect_SIM33ELA.kicad_sch (KiCad schematic)
At the start: 69 parts, among them J1 U.FL-R-SMT_10_, J2 MICROQTJ, Q1 DTC143ZUAT106, Q2 DTC143ZUAT106, Q3 AO3415, Q4 BSS138, Q5 BSS138, Q6 BSS138, U1 ESP32-C3FH4, U2 SIM33ELA, U3 TP4057, U4 EG800KEULC-I03-SNNSA, U5 DIODES AP2210N-3.3TRG1

Commit message: ultima version
Parts:
- removed D2, D3, D4: KUU SS36, Diode_SMD:D_SOD-123F, symbol Snapeda:KUU SS36
- added D2, D3, D4: D_Shockley, Diode_SMD:D_SOD-123F, symbol Device:D_Shockley
- added D6, D7: LED, LED_SMD:LED_0603_1608Metric_Pad1.05x0.95mm_HandSolder, symbol Device:LED
- added Q4, Q5: DTC143ZUAT106, Package_TO_SOT_SMD:SOT-323_SC-70, symbol Transistor_BJT:DTC143Z
- added R16, R17: 2.2k, Resistor_SMD:R_0603_1608Metric_Pad0.98x0.95mm_HandSolder, symbol Device:R_Small
- C14: renamed from C11; price 0.0567 -> 0.0688
- C16: renamed from C13; link (none) -> https://www.lcsc.com/product-detail/C77085.html?s_z=n_murat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; part number (none) -> GRM31CR60J107ME39L
- C17: renamed from C14; link (none) -> https://www.lcsc.com/product-detail/C77085.html?s_z=n_murat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; part number (none) -> GRM31CR60J107ME39L
- C18: renamed from C15; link (none) -> https://www.lcsc.com/product-detail/C77085.html?s_z=n_murat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; part number (none) -> GRM31CR60J107ME39L
- C19: renamed from C16; link (none) -> https://www.lcsc.com/product-detail/C77085.html?s_z=n_murat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; part number (none) -> GRM31CR60J107ME39L
- C20: renamed from C17; link (none) -> https://www.lcsc.com/product-detail/C77085.html?s_z=n_murat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; part number (none) -> GRM31CR60J107ME39L
- C21: renamed from C18; manufacturer (none) -> murata
- NANO-SIM-0501A-P1: Link https://www.lcsc.com/product-detail/C29780392.html?s_z=n_NA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 -> (none); link (none) -> https://www.lcsc.com/product-detail/C29780392.html?s_z=n_NA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
- Q1, Q2: link (none) -> https://www.lcsc.com/product-detail/C190246.html
- Q3: Link https://www.lcsc.com/product-detail/C5350989.html -> (none); link (none) -> https://www.lcsc.com/product-detail/C5350989.html
- U1: link (none) -> https://www.lcsc.com/product-detail/C2858491.html?s_z=n_ESP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
- U3: link (none) -> https://www.lcsc.com/product-detail/C725791.html?s_z=n_TP40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
- U4: link (none) -> https://es.aliexpress.com/item/1005009420162459.html?spm=a2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
- renumbered C7 to C10, C8 to C11, C9 to C12, C10 to C13, C12 to C15, C25 to C2, C19 to C22, C20 to C23, C21 to C24, C22 to C25, C23 to C26, C24 to C27, C2 to C3, C26 to C4, C27 to C5, C3 to C6, C4 to C7, C5 to C8, C6 to C9, Q4 to Q6, Q5 to Q7, Q6 to Q8, R9 to R10, R10 to R11, R11 to R12, R12 to R13, R13 to R14, R18 to R15, R14 to R18, R15 to R19, R16 to R20, R17 to R4, R4 to R5, R5 to R6, R6 to R7, R7 to R8, R8 to R9
Connections:
- net +4V: now also D4.1 (K)
- net +5V: now also D2.2 (A)
- net EG800K.VBAT: now also D6.2 (A), D7.2 (A)
- net GND: now also U2.4 (GND), U2.5 (GND), Q4.2 (E), Q5.2 (E)
- net EG800K.NET_STATUS: now reaches U4.16 (NET_STATUS)
- net EG800K.NET_STATUS: now also Q5.1 (B)
- net EG800K.STATUS: now reaches U4.25 (STATUS)
- net EG800K.STATUS: now also Q4.1 (B)
- new net: Q4.3 (C), R16.1
- new net: Q5.3 (C), R17.1
- new net: D7.1 (K), R17.2
- new net: D3.1 (K), D4.2 (A)
- new net: D2.1 (K), D3.2 (A)
- new net: D6.1 (K), R16.2
