File: EG800K-LA-devboard.kicad_pcb (KiCad board)
At the start: 4 copper layers, 35 x 35 mm, 46 parts, among them J1 U.FL-R-SMT_10_, J2 MICROQTJ, J4 Conn_01x11_Pin, Q1 DTC143ZUAT106, Q2 DTC143ZUAT106, Q4 DTC143ZUAT106, Q5 DTC143ZUAT106, U1 EG800KEULC-I03-SNNSA

Commit message: cambio de etiquetas
Parts:
- added kibuzzard-6A78147A: G***, kibuzzard-6A78147A, F.Cu at (150.0, 68.1)
- added kibuzzard-6A781493: G***, kibuzzard-6A781493, F.Cu at (150.0, 73.2)
- added kibuzzard-6A7814A6: G***, kibuzzard-6A7814A6, F.Cu at (150.1, 78.2)
- added kibuzzard-6A7814D1: G***, kibuzzard-6A7814D1, F.Cu at (150.0, 75.7)
- added kibuzzard-6A7814E0: G***, kibuzzard-6A7814E0, F.Cu at (150.0, 70.6)
- added kibuzzard-6A7814F3: G***, kibuzzard-6A7814F3, F.Cu at (150.0, 65.5)
- added kibuzzard-6A781522: G***, kibuzzard-6A781522, F.Cu at (150.0, 80.8)
- added kibuzzard-6A78152D: G***, kibuzzard-6A78152D, F.Cu at (150.0, 83.3)
- added kibuzzard-6A781536: G***, kibuzzard-6A781536, F.Cu at (150.0, 85.9)
Other:
- board text removed: "5V+"
- board text removed: "EG800.RDX"
- board text removed: "EG800.RI"
- board text removed: "EG800.TXD"
- board text removed: "EG800K.DTR"
- board text removed: "PWRKEY"
- board text removed: "RESET"
- board text removed: "V_EXT 1.8v"
- board text removed: "vBAT (3.7v)"
